Commit message: refactor

File: src/husky_kinova_sim/description/kinova_gen3.xacro (robot description, xacro)
@@ -113,5 +113,5 @@
     <child link="forearm_link" />
     <axis xyz="0 0 1" />
-    <limit lower="-2.57" upper="2.57" effort="39" velocity="1.3963" acceleration="1.0"/>  <!-- Added acceleration limit -->
+    <limit effort="39" velocity="1.3963" acceleration="1.0"/>  <!-- Added acceleration limit -->
   </joint>
   <link name="spherical_wrist_1_link">
