Commit message: update mesh file paths to use package:// format for consistency

File: src/husky_kinova_sim/description/husky_core.xacro (robot description, xacro)
@@ -26,5 +26,6 @@
       <!--<origin rpy="0 0 0" xyz="0 0 0"/>-->
       <geometry>
-        <mesh filename="file://$(find husky_bringup)/meshes/base_link.STL"/>
+        <!--<mesh filename="package://husky_kinova_sim/meshes/base_link.STL"/>-->
+        <mesh filename="package://husky_kinova_sim/meshes/base_link.STL"/>
       </geometry>
       <material name="Black"/>
@@ -33,5 +34,5 @@
       <!--<origin rpy="0 0 0" xyz="0 0 0"/>-->
       <geometry>
-        <mesh filename="file://$(find husky_bringup)/meshes/base_link.STL"/>
+        <mesh filename="package://husky_kinova_sim/meshes/base_link.STL"/>
         <!--<box size="0.515 0.515 0.1"/>-->
       </geometry>
@@ -61,5 +62,5 @@
         <origin rpy="0 0 0" xyz="0 0 0"/>
         <geometry>
-          <mesh filename="file://$(find husky_bringup)/meshes/wheel.STL"/>
+          <mesh filename="package://husky_kinova_sim/meshes/wheel.STL"/>
         </geometry>
         <material name="DarkGrey"/>
@@ -68,5 +69,5 @@
         <origin rpy="1.57079633 0 0" xyz="0 0 0"/>
         <geometry>
-          <!--<mesh filename="file://$(find husky_bringup)/meshes/wheel.STL"/> -->
+          <!--<mesh filename="package://husky_kinova_sim/meshes/wheel.STL"/> -->
           <cylinder radius="0.165" length="0.12"/>
         </geometry>
@@ -106,5 +107,5 @@
     <visual>
       <geometry>
-        <mesh filename="file://$(find husky_bringup)/meshes/top_plate.STL"/>
+        <mesh filename="package://husky_kinova_sim/meshes/top_plate.STL"/>
       </geometry>
       <material name="Yellow"/>
@@ -113,5 +114,5 @@
       <origin rpy="0 0 0" xyz="0 0 0"/>
        <geometry>
-        <mesh filename="file://$(find husky_bringup)/meshes/top_plate.STL"/>
+        <mesh filename="package://husky_kinova_sim/meshes/top_plate.STL"/>
        </geometry>
     </collision>
@@ -125,12 +126,12 @@
     <visual>
       <geometry>
-        <mesh filename="file://$(find husky_bringup)/meshes/user_rail.STL"/>
-      </geometry>
-      <material name="DarkGrey"/>
-    </visual>
-    <collision>
-      <origin rpy="0 0 0" xyz="0 0 0"/>
-       <geometry>
-        <mesh filename="file://$(find husky_bringup)/meshes/user_rail.STL"/>
+        <mesh filename="package://husky_kinova_sim/meshes/user_rail.STL"/>
+      </geometry>
+      <material name="DarkGrey"/>
+    </visual>
+    <collision>
+      <origin rpy="0 0 0" xyz="0 0 0"/>
+       <geometry>
+        <mesh filename="package://husky_kinova_sim/meshes/user_rail.STL"/>
        </geometry>
     </collision>
@@ -145,12 +146,12 @@
     <visual>
       <geometry>
-        <mesh filename="file://$(find husky_bringup)/meshes/bumper.STL"/>
-      </geometry>
-      <material name="DarkGrey"/>
-    </visual>
-    <collision>
-      <origin rpy="0 0 0" xyz="0 0 0"/>
-       <geometry>
-        <mesh filename="file://$(find husky_bringup)/meshes/bumper.STL"/>
+        <mesh filename="package://husky_kinova_sim/meshes/bumper.STL"/>
+      </geometry>
+      <material name="DarkGrey"/>
+    </visual>
+    <collision>
+      <origin rpy="0 0 0" xyz="0 0 0"/>
+       <geometry>
+        <mesh filename="package://husky_kinova_sim/meshes/bumper.STL"/>
        </geometry>
     </collision>
@@ -165,12 +166,12 @@
     <visual>
       <geometry>
-        <mesh filename="file://$(find husky_bringup)/meshes/bumper.STL"/>
-      </geometry>
-      <material name="DarkGrey"/>
-    </visual>
-    <collision>
-      <origin rpy="0 0 0" xyz="0 0 0"/>
-       <geometry>
-        <mesh filename="file://$(find husky_bringup)/meshes/bumper.STL"/>
+        <mesh filename="package://husky_kinova_sim/meshes/bumper.STL"/>
+      </geometry>
+      <material name="DarkGrey"/>
+    </visual>
+    <collision>
+      <origin rpy="0 0 0" xyz="0 0 0"/>
+       <geometry>
+        <mesh filename="package://husky_kinova_sim/meshes/bumper.STL"/>
        </geometry>
     </collision>
@@ -185,12 +186,12 @@
     <visual>
       <geometry>
-        <mesh filename="file://$(find husky_bringup)/meshes/payload_plate.STL"/>
-      </geometry>
-      <material name="DarkGrey"/>
-    </visual>
-    <collision>
-      <origin rpy="0 0 0" xyz="0 0 0"/>
-       <geometry>
-         <mesh filename="file://$(find husky_bringup)/meshes/payload_plate.STL"/>
+        <mesh filename="package://husky_kinova_sim/meshes/payload_plate.STL"/>
+      </geometry>
+      <material name="DarkGrey"/>
+    </visual>
+    <collision>
+      <origin rpy="0 0 0" xyz="0 0 0"/>
+       <geometry>
+         <mesh filename="package://husky_kinova_sim/meshes/payload_plate.STL"/>
       </geometry>
     </collision>
@@ -206,5 +207,5 @@
       <origin rpy="0 0 3.14159265" xyz="0 0 0"/>
       <geometry>
-        <mesh filename="file://$(find husky_bringup)/meshes/510_mm_sensor_arch.STL"/>
+        <mesh filename="package://husky_kinova_sim/meshes/510_mm_sensor_arch.STL"/>
       </geometry>
       <material name="DarkGrey"/>
@@ -213,5 +214,5 @@
       <origin rpy="0 0 3.14159265" xyz="0 0 0"/>
       <geometry>
-        <mesh filename="file://$(find husky_bringup)/meshes/510_mm_sensor_arch.STL"/>
+        <mesh filename="package://husky_kinova_sim/meshes/510_mm_sensor_arch.STL"/>
       </geometry>
     </collision>

File: src/husky_kinova_sim/description/kinova_gen3.xacro (robot description, xacro)
@@ -10,14 +10,14 @@
       <origin xyz="0 0 0" rpy="0 0 0" />
       <geometry>
-        <mesh filename="file://$(find husky_bringup)/meshes/kinova/arm_base.STL" />
-      </geometry>
-      <material name="">
-        <color rgba="0.75294 0.75294 0.75294 1" />
-      </material>
-    </visual>
-    <collision>
-      <origin xyz="0 0 0" rpy="0 0 0" />
-      <geometry>
-        <mesh filename="file://$(find husky_bringup)/meshes/kinova/arm_base.STL" />
+        <mesh filename="package://husky_kinova_sim/meshes/kinova/arm_base.STL" />
+      </geometry>
+      <material name="">
+        <color rgba="0.75294 0.75294 0.75294 1" />
+      </material>
+    </visual>
+    <collision>
+      <origin xyz="0 0 0" rpy="0 0 0" />
+      <geometry>
+        <mesh filename="package://husky_kinova_sim/meshes/kinova/arm_base.STL" />
       </geometry>
     </collision>
@@ -37,14 +37,14 @@
       <origin xyz="0 0 0" rpy="0 0 0" />
       <geometry>
-        <mesh filename="file://$(find husky_bringup)/meshes/kinova/shoulder_link.STL" />
-      </geometry>
-      <material name="">
-        <color rgba="0.75294 0.75294 0.75294 1" />
-      </material>
-    </visual>
-    <collision>
-      <origin xyz="0 0 0" rpy="0 0 0" />
-      <geometry>
-        <mesh filename="file://$(find husky_bringup)/meshes/kinova/shoulder_link.STL" />
+        <mesh filename="package://husky_kinova_sim/meshes/kinova/shoulder_link.STL" />
+      </geometry>
+      <material name="">
+        <color rgba="0.75294 0.75294 0.75294 1" />
+      </material>
+    </visual>
+    <collision>
+      <origin xyz="0 0 0" rpy="0 0 0" />
+      <geometry>
+        <mesh filename="package://husky_kinova_sim/meshes/kinova/shoulder_link.STL" />
       </geometry>
     </collision>
@@ -66,14 +66,14 @@
       <origin xyz="0 0 0" rpy="0 0 0" />
       <geometry>
-        <mesh filename="file://$(find husky_bringup)/meshes/kinova/bicep_link.STL" />
-      </geometry>
-      <material name="">
-        <color rgba="0.75294 0.75294 0.75294 1" />
-      </material>
-    </visual>
-    <collision>
-      <origin xyz="0 0 0" rpy="0 0 0" />
-      <geometry>
-        <mesh filename="file://$(find husky_bringup)/meshes/kinova/bicep_link.STL" />
+        <mesh filename="package://husky_kinova_sim/meshes/kinova/bicep_link.STL" />
+      </geometry>
+      <material name="">
+        <color rgba="0.75294 0.75294 0.75294 1" />
+      </material>
+    </visual>
+    <collision>
+      <origin xyz="0 0 0" rpy="0 0 0" />
+      <geometry>
+        <mesh filename="package://husky_kinova_sim/meshes/kinova/bicep_link.STL" />
       </geometry>
     </collision>
@@ -95,14 +95,14 @@
       <origin xyz="0 0 0" rpy="0 0 0" />
       <geometry>
-        <mesh filename="file://$(find husky_bringup)/meshes/kinova/forearm_link.STL" />
-      </geometry>
-      <material name="">
-        <color rgba="0.75294 0.75294 0.75294 1" />
-      </material>
-    </visual>
-    <collision>
-      <origin xyz="0 0 0" rpy="0 0 0" />
-      <geometry>
-        <mesh filename="file://$(find husky_bringup)/meshes/kinova/forearm_link.STL" />
+        <mesh filename="package://husky_kinova_sim/meshes/kinova/forearm_link.STL" />
+      </geometry>
+      <material name="">
+        <color rgba="0.75294 0.75294 0.75294 1" />
+      </material>
+    </visual>
+    <collision>
+      <origin xyz="0 0 0" rpy="0 0 0" />
+      <geometry>
+        <mesh filename="package://husky_kinova_sim/meshes/kinova/forearm_link.STL" />
       </geometry>
     </collision>
@@ -124,14 +124,14 @@
       <origin xyz="0 0 0" rpy="0 0 0" />
       <geometry>
-        <mesh filename="file://$(find husky_bringup)/meshes/kinova/spherical_wrist_1_link.STL" />
-      </geometry>
-      <material name="">
-        <color rgba="0.75294 0.75294 0.75294 1" />
-      </material>
-    </visual>
-    <collision>
-      <origin xyz="0 0 0" rpy="0 0 0" />
-      <geometry>
-        <mesh filename="file://$(find husky_bringup)/meshes/kinova/spherical_wrist_1_link.STL" />
+        <mesh filename="package://husky_kinova_sim/meshes/kinova/spherical_wrist_1_link.STL" />
+      </geometry>
+      <material name="">
+        <color rgba="0.75294 0.75294 0.75294 1" />
+      </material>
+    </visual>
+    <collision>
+      <origin xyz="0 0 0" rpy="0 0 0" />
+      <geometry>
+        <mesh filename="package://husky_kinova_sim/meshes/kinova/spherical_wrist_1_link.STL" />
       </geometry>
     </collision>
@@ -153,14 +153,14 @@
       <origin xyz="0 0 0" rpy="0 0 0" />
       <geometry>
-        <mesh filename="file://$(find husky_bringup)/meshes/kinova/spherical_wrist_2_link.STL" />
-      </geometry>
-      <material name="">
-        <color rgba="0.75294 0.75294 0.75294 1" />
-      </material>
-    </visual>
-    <collision>
-      <origin xyz="0 0 0" rpy="0 0 0" />
-      <geometry>
-        <mesh filename="file://$(find husky_bringup)/meshes/kinova/spherical_wrist_2_link.STL" />
+        <mesh filename="package://husky_kinova_sim/meshes/kinova/spherical_wrist_2_link.STL" />
+      </geometry>
+      <material name="">
+        <color rgba="0.75294 0.75294 0.75294 1" />
+      </material>
+    </visual>
+    <collision>
+      <origin xyz="0 0 0" rpy="0 0 0" />
+      <geometry>
+        <mesh filename="package://husky_kinova_sim/meshes/kinova/spherical_wrist_2_link.STL" />
       </geometry>
     </collision>
@@ -182,14 +182,14 @@
       <origin xyz="0 0 0" rpy="0 0 0" />
       <geometry>
-        <mesh filename="file://$(find husky_bringup)/meshes/kinova/bracelet_with_vision_link.STL" />
-      </geometry>
-      <material name="">
-        <color rgba="0.75294 0.75294 0.75294 1" />
-      </material>
-    </visual>
-    <collision>
-      <origin xyz="0 0 0" rpy="0 0 0" />
-      <geometry>
-        <mesh filename="file://$(find husky_bringup)/meshes/kinova/bracelet_with_vision_link.STL" />
+        <mesh filename="package://husky_kinova_sim/meshes/kinova/bracelet_with_vision_link.STL" />
+      </geometry>
+      <material name="">
+        <color rgba="0.75294 0.75294 0.75294 1" />
+      </material>
+    </visual>
+    <collision>
+      <origin xyz="0 0 0" rpy="0 0 0" />
+      <geometry>
+        <mesh filename="package://husky_kinova_sim/meshes/kinova/bracelet_with_vision_link.STL" />
       </geometry>
     </collision>

File: src/husky_kinova_sim/description/omni_60.xacro (robot description, xacro)
@@ -6,5 +6,5 @@
       <origin xyz="0 0 0" rpy="0 3.14159265 1.57079633"/>
       <geometry>
-        <mesh filename="file://$(find husky_bringup)/meshes/omni_60.STL"/>
+        <mesh filename="package://husky_kinova_sim/meshes/omni_60.STL"/>
       </geometry>
       <material name="Blue"/>
@@ -13,5 +13,5 @@
       <origin xyz="0 0 0" rpy="0 3.14159265 1.57079633"/>
       <geometry>
-        <mesh filename="file://$(find husky_bringup)/meshes/omni_60.STL"/>
+        <mesh filename="package://husky_kinova_sim/meshes/omni_60.STL"/>
       </geometry>
     </collision>

File: src/husky_kinova_sim/description/velodyne_v16.xacro (robot description, xacro)
@@ -3,5 +3,5 @@
 <!-- NOT MINE. FROM https://github.com/ToyotaResearchInstitute/velodyne_simulator.git -->
 <!--##################################################################################-->
-<robot xmlns:xacro="http://www.ros.org/wiki/xacro"> <!-- Changed robot name for clarity -->
+<robot xmlns:xacro="http://www.ros.org/wiki/xacro">
   <xacro:property name="M_PI" value="3.1415926535897931"/>
   <!-- Default parameters for the VLP-16 sensor -->
@@ -37,10 +37,10 @@
     <visual>
       <geometry>
-        <mesh filename="file://$(find husky_bringup)/meshes/velodyne_v16/VLP16_base_1.dae"/>
+        <mesh filename="package://husky_kinova_sim/meshes/velodyne_v16/VLP16_base_1.dae"/>
       </geometry>
     </visual>
     <visual>
       <geometry>
-        <mesh filename="file://$(find husky_bringup)/meshes/velodyne_v16/VLP16_base_2.dae"/>
+        <mesh filename="package://husky_kinova_sim/meshes/velodyne_v16/VLP16_base_2.dae"/>
       </geometry>
     </visual>
@@ -66,5 +66,5 @@
       <origin xyz="0 0 -0.0377"/> <!-- Adjust visual origin to match mesh -->
       <geometry>
-        <mesh filename="file://$(find husky_bringup)/meshes/velodyne_v16/VLP16_scan.dae"/>
+        <mesh filename="package://husky_kinova_sim/meshes/velodyne_v16/VLP16_scan.dae"/>
       </geometry>
     </visual>
@@ -72,5 +72,5 @@
       <origin xyz="0 0 -0.0377"/>
       <geometry>
-        <mesh filename="file://$(find husky_bringup)/meshes/velodyne_v16/VLP16_scan.dae"/>
+        <mesh filename="package://husky_kinova_sim/meshes/velodyne_v16/VLP16_scan.dae"/>
       </geometry>
     </collision>
