Commit message: Refactor code structure for improved readability and maintainability

File: src/husky_kinova_sim/description/husky_core.xacro (robot description, xacro)
@@ -26,6 +26,5 @@
       <!--<origin rpy="0 0 0" xyz="0 0 0"/>-->
       <geometry>
-        <!--<mesh filename="file://$(find husky_bringup)/meshes/base_link.STL"/>-->
-        <mesh filename="file://$(find husky_bringup)/meshes/base_link.STL"/>
+        <mesh filename="file://$(find husky_kinova_sim)/meshes/base_link.STL"/>
       </geometry>
       <material name="Black"/>
@@ -34,5 +33,5 @@
       <!--<origin rpy="0 0 0" xyz="0 0 0"/>-->
       <geometry>
-        <mesh filename="file://$(find husky_bringup)/meshes/base_link.STL"/>
+        <mesh filename="file://$(find husky_kinova_sim)/meshes/base_link.STL"/>
         <!--<box size="0.515 0.515 0.1"/>-->
       </geometry>
@@ -62,5 +61,5 @@
         <origin rpy="0 0 0" xyz="0 0 0"/>
         <geometry>
-          <mesh filename="file://$(find husky_bringup)/meshes/wheel.STL"/>
+          <mesh filename="file://$(find husky_kinova_sim)/meshes/wheel.STL"/>
         </geometry>
         <material name="DarkGrey"/>
@@ -69,5 +68,5 @@
         <origin rpy="1.57079633 0 0" xyz="0 0 0"/>
         <geometry>
-          <!--<mesh filename="file://$(find husky_bringup)/meshes/wheel.STL"/> -->
+          <!--<mesh filename="file://$(find husky_kinova_sim)/meshes/wheel.STL"/> -->
           <cylinder radius="0.165" length="0.12"/>
         </geometry>
@@ -107,5 +106,5 @@
     <visual>
       <geometry>
-        <mesh filename="file://$(find husky_bringup)/meshes/top_plate.STL"/>
+        <mesh filename="file://$(find husky_kinova_sim)/meshes/top_plate.STL"/>
       </geometry>
       <material name="Yellow"/>
@@ -114,5 +113,5 @@
       <origin rpy="0 0 0" xyz="0 0 0"/>
        <geometry>
-        <mesh filename="file://$(find husky_bringup)/meshes/top_plate.STL"/>
+        <mesh filename="file://$(find husky_kinova_sim)/meshes/top_plate.STL"/>
        </geometry>
     </collision>
@@ -126,12 +125,12 @@
     <visual>
       <geometry>
-        <mesh filename="file://$(find husky_bringup)/meshes/user_rail.STL"/>
-      </geometry>
-      <material name="DarkGrey"/>
-    </visual>
-    <collision>
-      <origin rpy="0 0 0" xyz="0 0 0"/>
-       <geometry>
-        <mesh filename="file://$(find husky_bringup)/meshes/user_rail.STL"/>
+        <mesh filename="file://$(find husky_kinova_sim)/meshes/user_rail.STL"/>
+      </geometry>
+      <material name="DarkGrey"/>
+    </visual>
+    <collision>
+      <origin rpy="0 0 0" xyz="0 0 0"/>
+       <geometry>
+        <mesh filename="file://$(find husky_kinova_sim)/meshes/user_rail.STL"/>
        </geometry>
     </collision>
@@ -146,12 +145,12 @@
     <visual>
       <geometry>
-        <mesh filename="file://$(find husky_bringup)/meshes/bumper.STL"/>
-      </geometry>
-      <material name="DarkGrey"/>
-    </visual>
-    <collision>
-      <origin rpy="0 0 0" xyz="0 0 0"/>
-       <geometry>
-        <mesh filename="file://$(find husky_bringup)/meshes/bumper.STL"/>
+        <mesh filename="file://$(find husky_kinova_sim)/meshes/bumper.STL"/>
+      </geometry>
+      <material name="DarkGrey"/>
+    </visual>
+    <collision>
+      <origin rpy="0 0 0" xyz="0 0 0"/>
+       <geometry>
+        <mesh filename="file://$(find husky_kinova_sim)/meshes/bumper.STL"/>
        </geometry>
     </collision>
@@ -166,12 +165,12 @@
     <visual>
       <geometry>
-        <mesh filename="file://$(find husky_bringup)/meshes/bumper.STL"/>
-      </geometry>
-      <material name="DarkGrey"/>
-    </visual>
-    <collision>
-      <origin rpy="0 0 0" xyz="0 0 0"/>
-       <geometry>
-        <mesh filename="file://$(find husky_bringup)/meshes/bumper.STL"/>
+        <mesh filename="file://$(find husky_kinova_sim)/meshes/bumper.STL"/>
+      </geometry>
+      <material name="DarkGrey"/>
+    </visual>
+    <collision>
+      <origin rpy="0 0 0" xyz="0 0 0"/>
+       <geometry>
+        <mesh filename="file://$(find husky_kinova_sim)/meshes/bumper.STL"/>
        </geometry>
     </collision>
@@ -186,12 +185,12 @@
     <visual>
       <geometry>
-        <mesh filename="file://$(find husky_bringup)/meshes/payload_plate.STL"/>
-      </geometry>
-      <material name="DarkGrey"/>
-    </visual>
-    <collision>
-      <origin rpy="0 0 0" xyz="0 0 0"/>
-       <geometry>
-         <mesh filename="file://$(find husky_bringup)/meshes/payload_plate.STL"/>
+        <mesh filename="file://$(find husky_kinova_sim)/meshes/payload_plate.STL"/>
+      </geometry>
+      <material name="DarkGrey"/>
+    </visual>
+    <collision>
+      <origin rpy="0 0 0" xyz="0 0 0"/>
+       <geometry>
+         <mesh filename="file://$(find husky_kinova_sim)/meshes/payload_plate.STL"/>
       </geometry>
     </collision>
@@ -207,5 +206,5 @@
       <origin rpy="0 0 3.14159265" xyz="0 0 0"/>
       <geometry>
-        <mesh filename="file://$(find husky_bringup)/meshes/510_mm_sensor_arch.STL"/>
+        <mesh filename="file://$(find husky_kinova_sim)/meshes/510_mm_sensor_arch.STL"/>
       </geometry>
       <material name="DarkGrey"/>
@@ -214,5 +213,5 @@
       <origin rpy="0 0 3.14159265" xyz="0 0 0"/>
       <geometry>
-        <mesh filename="file://$(find husky_bringup)/meshes/510_mm_sensor_arch.STL"/>
+        <mesh filename="file://$(find husky_kinova_sim)/meshes/510_mm_sensor_arch.STL"/>
       </geometry>
     </collision>

File: src/husky_kinova_sim/description/kinova_gen3.xacro (robot description, xacro)
@@ -10,14 +10,14 @@
       <origin xyz="0 0 0" rpy="0 0 0" />
       <geometry>
-        <mesh filename="file://$(find husky_bringup)/meshes/kinova/arm_base.STL" />
-      </geometry>
-      <material name="">
-        <color rgba="0.75294 0.75294 0.75294 1" />
-      </material>
-    </visual>
-    <collision>
-      <origin xyz="0 0 0" rpy="0 0 0" />
-      <geometry>
-        <mesh filename="file://$(find husky_bringup)/meshes/kinova/arm_base.STL" />
+        <mesh filename="file://$(find husky_kinova_sim)/meshes/kinova/arm_base.STL" />
+      </geometry>
+      <material name="">
+        <color rgba="0.75294 0.75294 0.75294 1" />
+      </material>
+    </visual>
+    <collision>
+      <origin xyz="0 0 0" rpy="0 0 0" />
+      <geometry>
+        <mesh filename="file://$(find husky_kinova_sim)/meshes/kinova/arm_base.STL" />
       </geometry>
     </collision>
@@ -37,14 +37,14 @@
       <origin xyz="0 0 0" rpy="0 0 0" />
       <geometry>
-        <mesh filename="file://$(find husky_bringup)/meshes/kinova/shoulder_link.STL" />
-      </geometry>
-      <material name="">
-        <color rgba="0.75294 0.75294 0.75294 1" />
-      </material>
-    </visual>
-    <collision>
-      <origin xyz="0 0 0" rpy="0 0 0" />
-      <geometry>
-        <mesh filename="file://$(find husky_bringup)/meshes/kinova/shoulder_link.STL" />
+        <mesh filename="file://$(find husky_kinova_sim)/meshes/kinova/shoulder_link.STL" />
+      </geometry>
+      <material name="">
+        <color rgba="0.75294 0.75294 0.75294 1" />
+      </material>
+    </visual>
+    <collision>
+      <origin xyz="0 0 0" rpy="0 0 0" />
+      <geometry>
+        <mesh filename="file://$(find husky_kinova_sim)/meshes/kinova/shoulder_link.STL" />
       </geometry>
     </collision>
@@ -66,14 +66,14 @@
       <origin xyz="0 0 0" rpy="0 0 0" />
       <geometry>
-        <mesh filename="file://$(find husky_bringup)/meshes/kinova/bicep_link.STL" />
-      </geometry>
-      <material name="">
-        <color rgba="0.75294 0.75294 0.75294 1" />
-      </material>
-    </visual>
-    <collision>
-      <origin xyz="0 0 0" rpy="0 0 0" />
-      <geometry>
-        <mesh filename="file://$(find husky_bringup)/meshes/kinova/bicep_link.STL" />
+        <mesh filename="file://$(find husky_kinova_sim)/meshes/kinova/bicep_link.STL" />
+      </geometry>
+      <material name="">
+        <color rgba="0.75294 0.75294 0.75294 1" />
+      </material>
+    </visual>
+    <collision>
+      <origin xyz="0 0 0" rpy="0 0 0" />
+      <geometry>
+        <mesh filename="file://$(find husky_kinova_sim)/meshes/kinova/bicep_link.STL" />
       </geometry>
     </collision>
@@ -95,14 +95,14 @@
       <origin xyz="0 0 0" rpy="0 0 0" />
       <geometry>
-        <mesh filename="file://$(find husky_bringup)/meshes/kinova/forearm_link.STL" />
-      </geometry>
-      <material name="">
-        <color rgba="0.75294 0.75294 0.75294 1" />
-      </material>
-    </visual>
-    <collision>
-      <origin xyz="0 0 0" rpy="0 0 0" />
-      <geometry>
-        <mesh filename="file://$(find husky_bringup)/meshes/kinova/forearm_link.STL" />
+        <mesh filename="file://$(find husky_kinova_sim)/meshes/kinova/forearm_link.STL" />
+      </geometry>
+      <material name="">
+        <color rgba="0.75294 0.75294 0.75294 1" />
+      </material>
+    </visual>
+    <collision>
+      <origin xyz="0 0 0" rpy="0 0 0" />
+      <geometry>
+        <mesh filename="file://$(find husky_kinova_sim)/meshes/kinova/forearm_link.STL" />
       </geometry>
     </collision>
@@ -113,5 +113,5 @@
     <child link="forearm_link" />
     <axis xyz="0 0 1" />
-    <limit effort="39" velocity="1.3963" acceleration="1.0"/>  <!-- Added acceleration limit -->
+    <limit lower="-2.57" upper="2.57" effort="39" velocity="1.3963" acceleration="1.0"/>  <!-- Added acceleration limit -->
   </joint>
   <link name="spherical_wrist_1_link">
@@ -124,14 +124,14 @@
       <origin xyz="0 0 0" rpy="0 0 0" />
       <geometry>
-        <mesh filename="file://$(find husky_bringup)/meshes/kinova/spherical_wrist_1_link.STL" />
-      </geometry>
-      <material name="">
-        <color rgba="0.75294 0.75294 0.75294 1" />
-      </material>
-    </visual>
-    <collision>
-      <origin xyz="0 0 0" rpy="0 0 0" />
-      <geometry>
-        <mesh filename="file://$(find husky_bringup)/meshes/kinova/spherical_wrist_1_link.STL" />
+        <mesh filename="file://$(find husky_kinova_sim)/meshes/kinova/spherical_wrist_1_link.STL" />
+      </geometry>
+      <material name="">
+        <color rgba="0.75294 0.75294 0.75294 1" />
+      </material>
+    </visual>
+    <collision>
+      <origin xyz="0 0 0" rpy="0 0 0" />
+      <geometry>
+        <mesh filename="file://$(find husky_kinova_sim)/meshes/kinova/spherical_wrist_1_link.STL" />
       </geometry>
     </collision>
@@ -153,14 +153,14 @@
       <origin xyz="0 0 0" rpy="0 0 0" />
       <geometry>
-        <mesh filename="file://$(find husky_bringup)/meshes/kinova/spherical_wrist_2_link.STL" />
-      </geometry>
-      <material name="">
-        <color rgba="0.75294 0.75294 0.75294 1" />
-      </material>
-    </visual>
-    <collision>
-      <origin xyz="0 0 0" rpy="0 0 0" />
-      <geometry>
-        <mesh filename="file://$(find husky_bringup)/meshes/kinova/spherical_wrist_2_link.STL" />
+        <mesh filename="file://$(find husky_kinova_sim)/meshes/kinova/spherical_wrist_2_link.STL" />
+      </geometry>
+      <material name="">
+        <color rgba="0.75294 0.75294 0.75294 1" />
+      </material>
+    </visual>
+    <collision>
+      <origin xyz="0 0 0" rpy="0 0 0" />
+      <geometry>
+        <mesh filename="file://$(find husky_kinova_sim)/meshes/kinova/spherical_wrist_2_link.STL" />
       </geometry>
     </collision>
@@ -182,14 +182,14 @@
       <origin xyz="0 0 0" rpy="0 0 0" />
       <geometry>
-        <mesh filename="file://$(find husky_bringup)/meshes/kinova/bracelet_with_vision_link.STL" />
-      </geometry>
-      <material name="">
-        <color rgba="0.75294 0.75294 0.75294 1" />
-      </material>
-    </visual>
-    <collision>
-      <origin xyz="0 0 0" rpy="0 0 0" />
-      <geometry>
-        <mesh filename="file://$(find husky_bringup)/meshes/kinova/bracelet_with_vision_link.STL" />
+        <mesh filename="file://$(find husky_kinova_sim)/meshes/kinova/bracelet_with_vision_link.STL" />
+      </geometry>
+      <material name="">
+        <color rgba="0.75294 0.75294 0.75294 1" />
+      </material>
+    </visual>
+    <collision>
+      <origin xyz="0 0 0" rpy="0 0 0" />
+      <geometry>
+        <mesh filename="file://$(find husky_kinova_sim)/meshes/kinova/bracelet_with_vision_link.STL" />
       </geometry>
     </collision>

File: src/husky_kinova_sim/description/omni_60.xacro (robot description, xacro)
@@ -6,5 +6,5 @@
       <origin xyz="0 0 0" rpy="0 3.14159265 1.57079633"/>
       <geometry>
-        <mesh filename="file://$(find husky_bringup)/meshes/omni_60.STL"/>
+        <mesh filename="file://$(find husky_kinova_sim)/meshes/omni_60.STL"/>
       </geometry>
       <material name="Blue"/>
@@ -13,5 +13,5 @@
       <origin xyz="0 0 0" rpy="0 3.14159265 1.57079633"/>
       <geometry>
-        <mesh filename="file://$(find husky_bringup)/meshes/omni_60.STL"/>
+        <mesh filename="file://$(find husky_kinova_sim)/meshes/omni_60.STL"/>
       </geometry>
     </collision>

File: src/husky_kinova_sim/description/velodyne_v16.xacro (robot description, xacro)
@@ -3,5 +3,5 @@
 <!-- NOT MINE. FROM https://github.com/ToyotaResearchInstitute/velodyne_simulator.git -->
 <!--##################################################################################-->
-<robot xmlns:xacro="http://www.ros.org/wiki/xacro">
+<robot xmlns:xacro="http://www.ros.org/wiki/xacro"> <!-- Changed robot name for clarity -->
   <xacro:property name="M_PI" value="3.1415926535897931"/>
   <!-- Default parameters for the VLP-16 sensor -->
@@ -37,10 +37,10 @@
     <visual>
       <geometry>
-        <mesh filename="file://$(find husky_bringup)/meshes/velodyne_v16/VLP16_base_1.dae"/>
+        <mesh filename="file://$(find husky_kinova_sim)/meshes/velodyne_v16/VLP16_base_1.dae"/>
       </geometry>
     </visual>
     <visual>
       <geometry>
-        <mesh filename="file://$(find husky_bringup)/meshes/velodyne_v16/VLP16_base_2.dae"/>
+        <mesh filename="file://$(find husky_kinova_sim)/meshes/velodyne_v16/VLP16_base_2.dae"/>
       </geometry>
     </visual>
@@ -66,5 +66,5 @@
       <origin xyz="0 0 -0.0377"/> <!-- Adjust visual origin to match mesh -->
       <geometry>
-        <mesh filename="file://$(find husky_bringup)/meshes/velodyne_v16/VLP16_scan.dae"/>
+        <mesh filename="file://$(find husky_kinova_sim)/meshes/velodyne_v16/VLP16_scan.dae"/>
       </geometry>
     </visual>
@@ -72,5 +72,5 @@
       <origin xyz="0 0 -0.0377"/>
       <geometry>
-        <mesh filename="file://$(find husky_bringup)/meshes/velodyne_v16/VLP16_scan.dae"/>
+        <mesh filename="file://$(find husky_kinova_sim)/meshes/velodyne_v16/VLP16_scan.dae"/>
       </geometry>
     </collision>

File: src/kinova_arm/config/husky.urdf.xacro (robot description, xacro)
@@ -3,5 +3,5 @@
     <xacro:arg name="initial_positions_file" default="initial_positions.yaml" />
     <!-- Import husky urdf file -->
-    <xacro:include filename="$(find husky_bringup)/description/husky.urdf.xacro" />
+    <xacro:include filename="$(find husky_kinova_sim)/description/husky.urdf.xacro" />
     <!-- Import control_xacro -->
     <xacro:include filename="husky.ros2_control.xacro" />
